File: pcb/main board/main board.kicad_pcb (KiCad board)
At the start: 2 copper layers, 29 parts, among them Q1 IRF8714PBF, Q2 IRF8714PBF, U1 L298HN, U2 L298HN, U3 LM2596S-5, U4 MCP23017_SO, U6 LM3150MH

Commit message: Modified LM2596S to be a module.
Parts:
- removed A1: RaspberryPi_Pico, Module:RaspberryPi_Pico_Common_Unspecified
- removed A2: RaspberryPi_Pico_W, Module:RaspberryPi_Pico_W_SMD_HandSolder
- removed A3, A4, A5: Pololu_Breakout_A4988, Module:Pololu_Breakout-16_15.2x20.3mm
- removed D1, D10, D11, D12, D13, D14, D15, D16, D2, D3, D4, D5, D6, D7, D8, D9: 1N4007, Diode_THT:D_DO-41_SOD81_P10.16mm_Horizontal
- removed D17: 1N5824, Diode_THT:D_DO-201AD_P15.24mm_Horizontal
- removed Q1, Q2: IRF8714PBF, Package_SO:SOIC-8_3.9x4.9mm_P1.27mm
- removed U1, U2: L298HN, Package_TO_SOT_THT:TO-220-15_P2.54x2.54mm_StaggerOdd_Lead5.84mm_TabDown
- removed U3: LM2596S-5, Package_TO_SOT_SMD:TO-263-5_TabPin3
- removed U4: MCP23017_SO, Package_SO:SOIC-28W_7.5x17.9mm_P1.27mm
- removed U6: LM3150MH, Package_SO:HTSSOP-14-1EP_4.4x5mm_P0.65mm_EP3.4x5mm_Mask3x3.1mm

Commit message: Started Motors Wiring
Parts:
- added A1: RaspberryPi_Pico, Module:RaspberryPi_Pico_Common_Unspecified, F.Cu at (211.6, 206.6)
- added A2: RaspberryPi_Pico_W, Module:RaspberryPi_Pico_Common_Unspecified, F.Cu at (102.7, 202.7)
- added A3: Pololu_Breakout_A4988, Module:Pololu_Breakout-16_15.2x20.3mm, F.Cu at (371.3, 153.9)
- added A4: Pololu_Breakout_A4988, Module:Pololu_Breakout-16_15.2x20.3mm, F.Cu at (371.3, 178.9)
- added A5: Pololu_Breakout_A4988, Module:Pololu_Breakout-16_15.2x20.3mm, F.Cu at (371.3, 203.9)
- added C1: 100nF, Capacitor_THT:C_Disc_D4.3mm_W1.9mm_P5.00mm, F.Cu at (166.2, 174.4)
- added C10: 10uF, Capacitor_THT:CP_Radial_D5.0mm_P2.50mm, F.Cu at (277.1, 158.4)
- added C11: 10uF, Capacitor_THT:CP_Radial_D5.0mm_P2.50mm, F.Cu at (277.1, 164.9)
- added C12: 100nF, Capacitor_THT:C_Disc_D4.3mm_W1.9mm_P5.00mm, F.Cu at (247.5, 65.4)
- added C13: 120pF, Capacitor_THT:C_Disc_D4.3mm_W1.9mm_P5.00mm, F.Cu at (247.5, 68.8)
- added C14: 120uF, Capacitor_THT:CP_Radial_D10.0mm_P5.00mm, F.Cu at (278.5, 174.0)
- added C15: 100uF, Capacitor_THT:CP_Radial_D10.0mm_P5.00mm, F.Cu at (156.4, 154.3)
- added C16: 100uF, Capacitor_THT:CP_Radial_D10.0mm_P5.00mm, F.Cu at (156.4, 165.8)
- added C17: 100uF, Capacitor_THT:CP_Radial_D10.0mm_P5.00mm, F.Cu at (156.4, 177.4)
- added C2: 100nF, Capacitor_THT:C_Disc_D4.3mm_W1.9mm_P5.00mm, F.Cu at (166.2, 177.8)
- added C3: 100nF, Capacitor_THT:C_Disc_D4.3mm_W1.9mm_P5.00mm, F.Cu at (166.2, 181.3)
- added C4: 100nF, Capacitor_THT:C_Disc_D4.3mm_W1.9mm_P5.00mm, F.Cu at (166.2, 184.8)
- added C7: 470nF, Capacitor_THT:C_Disc_D4.3mm_W1.9mm_P5.00mm, F.Cu at (247.5, 55.0)
- added C8: 2.2uF, Capacitor_THT:C_Disc_D4.3mm_W1.9mm_P5.00mm, F.Cu at (247.5, 58.5)
- added C9: 15nF, Capacitor_THT:C_Disc_D4.3mm_W1.9mm_P5.00mm, F.Cu at (247.5, 62.0)
- added D1: 1N4007, Diode_THT:D_DO-41_SOD81_P10.16mm_Horizontal, F.Cu at (360.5, 28.3)
- added D10: 1N4007, Diode_THT:D_DO-41_SOD81_P10.16mm_Horizontal, F.Cu at (130.9, 141.2)
- added D11: 1N4007, Diode_THT:D_DO-41_SOD81_P10.16mm_Horizontal, F.Cu at (130.9, 145.5)
- added D12: 1N4007, Diode_THT:D_DO-41_SOD81_P10.16mm_Horizontal, F.Cu at (130.9, 149.7)
- added D13: 1N4007, Diode_THT:D_DO-41_SOD81_P10.16mm_Horizontal, F.Cu at (130.9, 154.0)
- added D14: 1N4007, Diode_THT:D_DO-41_SOD81_P10.16mm_Horizontal, F.Cu at (130.9, 158.2)
- added D15: 1N4007, Diode_THT:D_DO-41_SOD81_P10.16mm_Horizontal, F.Cu at (130.9, 162.5)
- added D16: 1N4007, Diode_THT:D_DO-41_SOD81_P10.16mm_Horizontal, F.Cu at (130.9, 166.7)
- added D2: 1N4007, Diode_THT:D_DO-41_SOD81_P10.16mm_Horizontal, F.Cu at (367.0, 28.3)
- added D3: 1N4007, Diode_THT:D_DO-41_SOD81_P10.16mm_Horizontal, F.Cu at (380.0, 28.3)
- added D4: 1N4007, Diode_THT:D_DO-41_SOD81_P10.16mm_Horizontal, F.Cu at (373.5, 28.3)
- added D5: 1N4007, Diode_THT:D_DO-41_SOD81_P10.16mm_Horizontal, F.Cu at (360.5, 49.0)
- added D6: 1N4007, Diode_THT:D_DO-41_SOD81_P10.16mm_Horizontal, F.Cu at (367.0, 49.0)
- added D7: 1N4007, Diode_THT:D_DO-41_SOD81_P10.16mm_Horizontal, F.Cu at (373.5, 49.0)
- added D8: 1N4007, Diode_THT:D_DO-41_SOD81_P10.16mm_Horizontal, F.Cu at (380.0, 49.0)
- added D9: 1N4007, Diode_THT:D_DO-41_SOD81_P10.16mm_Horizontal, F.Cu at (130.9, 137.0)
- added J1: Motor 0 Conn, Connector_PinHeader_2.54mm:PinHeader_1x02_P2.54mm_Vertical, F.Cu at (388.8, 38.5)
- added J10: 12V Battery, Connector_PinHeader_2.54mm:PinHeader_1x02_P2.54mm_Vertical, F.Cu at (269.2, 128.0)
- added J11: BAU, Connector_PinHeader_2.54mm:PinHeader_1x02_P2.54mm_Vertical, F.Cu at (269.2, 137.6)
- added J12: Servo 4 Conn, Connector_PinHeader_2.54mm:PinHeader_1x03_P2.54mm_Vertical, F.Cu at (245.8, 127.5)
- added J13: Servo 1 Conn, Connector_PinHeader_2.54mm:PinHeader_1x03_P2.54mm_Vertical, F.Cu at (245.8, 135.4)
- added J14: Servo 2 Conn, Connector_PinHeader_2.54mm:PinHeader_1x03_P2.54mm_Vertical, F.Cu at (245.8, 143.3)
- added J15: Servo 3 Conn, Connector_PinHeader_2.54mm:PinHeader_1x03_P2.54mm_Vertical, F.Cu at (245.8, 151.2)
- added J16: Servo 5 Conn, Connector_PinHeader_2.54mm:PinHeader_1x03_P2.54mm_Vertical, F.Cu at (245.8, 159.1)
- added J17: Servo 6 Conn, Connector_PinHeader_2.54mm:PinHeader_1x03_P2.54mm_Vertical, F.Cu at (245.8, 167.0)
- added J2: Motor 1 Conn, Connector_PinHeader_2.54mm:PinHeader_1x02_P2.54mm_Vertical, F.Cu at (388.8, 51.5)
- added J3: Motor 2 Conn, Connector_PinHeader_2.54mm:PinHeader_1x02_P2.54mm_Vertical, F.Cu at (146.0, 171.9)
- added J4: Motor 3 Conn, Connector_PinHeader_2.54mm:PinHeader_1x02_P2.54mm_Vertical, F.Cu at (146.0, 181.6)
- added J5: I2C 0 Conn, Connector_PinHeader_2.54mm:PinHeader_1x04_P2.54mm_Vertical, F.Cu at (250.1, 187.0)
- added J6: I2C 1 Conn, Connector_PinHeader_2.54mm:PinHeader_1x04_P2.54mm_Vertical, F.Cu at (270.1, 188.0)
- added J7: Stepper 0 Conn, Connector_PinHeader_2.54mm:PinHeader_1x04_P2.54mm_Vertical, F.Cu at (380.0, 148.8)
- added J8: Stepper 1 Conn, Connector_PinHeader_2.54mm:PinHeader_1x04_P2.54mm_Vertical, F.Cu at (380.0, 173.8)
- added J9: Stepper 2 Conn, Connector_PinHeader_2.54mm:PinHeader_1x04_P2.54mm_Vertical, F.Cu at (380.0, 198.8)
- added L2: 1.8uH, Inductor_SMD:L_APV_APH1040, F.Cu at (274.1, 149.3)
- added Q1: IRF8714PBF, Package_SO:SOIC-8_3.9x4.9mm_P1.27mm, F.Cu at (230.0, 37.5)
- added Q2: IRF8714PBF, Package_SO:SOIC-8_3.9x4.9mm_P1.27mm, F.Cu at (238.0, 37.5)
- added R1: 665Ω, Resistor_THT:R_Axial_DIN0207_L6.3mm_D2.5mm_P10.16mm_Horizontal, F.Cu at (254.8, 145.5)
- added R2: 82.5kΩ, Resistor_THT:R_Axial_DIN0207_L6.3mm_D2.5mm_P10.16mm_Horizontal, F.Cu at (254.8, 149.6)
- added R3: 73.2kΩ, Resistor_THT:R_Axial_DIN0207_L6.3mm_D2.5mm_P10.16mm_Horizontal, F.Cu at (254.8, 153.6)
- added R4: 10kΩ, Resistor_THT:R_Axial_DIN0207_L6.3mm_D2.5mm_P10.16mm_Horizontal, F.Cu at (254.8, 157.7)
- added U1: L298HN, Package_TO_SOT_THT:TO-220-15_P2.54x2.54mm_StaggerOdd_Lead5.84mm_TabDown, F.Cu at (352.8, 32.5)
- added U2: L298HN, Package_TO_SOT_THT:TO-220-15_P2.54x2.54mm_StaggerOdd_Lead5.84mm_TabDown, F.Cu at (320.7, 70.9)
- added U3: ~, LM2596S-Module:LM2596S-Module, F.Cu at (144.5, 62.0)
- added U4: MCP23017_SO, Package_SO:SOIC-28W_7.5x17.9mm_P1.27mm, F.Cu at (332.9, 98.8)
- added U6: LM3150MH, Package_SO:HTSSOP-14-1EP_4.4x5mm_P0.65mm_EP3.4x5mm_Mask3x3.1mm, F.Cu at (235.8, 51.9)
Routing:
- net Net-(D1-A): track 0.00 -> 64.6 mm
- net Net-(D3-A): track 0.00 -> 56.4 mm
- net Net-(D4-A): track 0.00 -> 47.4 mm
- net Net-(D2-A): track 0.00 -> 36.6 mm
Other:
- board outline added: 48 x 22 mm
